File: board_cad/novex_rasp_hat/novex_rasp_hat.kicad_pcb (KiCad board)
At the start: 4 copper layers, 65 x 30 mm, 16 parts, among them J1 GPIO, J2 USB_A

Commit message: CAD Novex Board Update v0.12
Parts:
- added ESP_USB: PinHeader_1x02_P1.27mm_Vertical, Connector_PinHeader_1.27mm:PinHeader_1x02_P1.27mm_Vertical, F.Cu at (108.8, 79.5)
- added U_MCU: TSSOP-20_4.4x6.5mm_P0.65mm, Package_SO:TSSOP-20_4.4x6.5mm_P0.65mm, F.Cu at (125.0, 82.8)
- added U_USBHUB: QFN-36-1EP_6x6mm_P0.5mm_EP3.7x3.7mm, Package_DFN_QFN:QFN-36-1EP_6x6mm_P0.5mm_EP3.7x3.7mm, F.Cu at (139.3, 82.7)
- added bat0+: SolderWire-0.127sqmm_1x01_D0.48mm_OD1mm, Connector_Wire:SolderWire-0.127sqmm_1x01_D0.48mm_OD1mm, F.Cu at (163.5, 91.8)
- added bat0-: SolderWire-0.127sqmm_1x01_D0.48mm_OD1mm, Connector_Wire:SolderWire-0.127sqmm_1x01_D0.48mm_OD1mm, F.Cu at (163.5, 89.0)
- added bat1+: SolderWire-0.127sqmm_1x01_D0.48mm_OD1mm, Connector_Wire:SolderWire-0.127sqmm_1x01_D0.48mm_OD1mm, F.Cu at (160.8, 91.8)
- added bat1-: SolderWire-0.127sqmm_1x01_D0.48mm_OD1mm, Connector_Wire:SolderWire-0.127sqmm_1x01_D0.48mm_OD1mm, F.Cu at (160.8, 89.0)
- esp_spi1: renamed from esp_spi; value PinSocket_2x06_P2.00mm_Horizontal -> Conn_02x06_Odd_Even
- lora0: value PinSocket_2x06_P2.00mm_Vertical -> Conn_02x06_Odd_Even
- moved D+ 0.45 mm to (139.5, 97.8)
- moved D- 0.45 mm to (141.0, 97.8)
- moved GND 0.45 mm to (142.5, 97.8)
- moved VBUS 0.45 mm to (138.0, 97.8)
- moved esp_spi1 0.35 mm to (121.2, 90.2)
- renumbered TP3 to D+, TP2 to D-, TP4 to GND, TP1 to VBUS
Connections:
- D+ pad 1: Net-(J2-D-) -> unconnected-(TP3-Pad1)
- D- pad 1: Net-(J2-D+) -> unconnected-(TP2-Pad1)
- GND pad 1: Net-(J2-GND) -> unconnected-(TP4-Pad1)
- J1 pad 11: /GPIO17 -> esp_rst
- J1 pad 13: /GPIO27 -> esp_boot
- J2 pad 1: Net-(J2-VBUS) -> unconnected-(J2-VBUS-Pad1)
- J2 pad 2: Net-(J2-D-) -> unconnected-(J2-D--Pad2)
- J2 pad 3: Net-(J2-D+) -> unconnected-(J2-D+-Pad3)
- J2 pad 4: Net-(J2-GND) -> unconnected-(J2-GND-Pad4)
- VBUS pad 1: Net-(J2-VBUS) -> unconnected-(TP1-Pad1)
- esp_comm1 pad 3: unconnected-(esp_comm1-Pin_3-Pad3) -> esp_boot
- esp_comm1 pad 4: unconnected-(esp_comm1-Pin_4-Pad4) -> esp_rst
- esp_spi1 pad 1: (no net) -> Net-(esp_spi1-Pin_1)
- esp_spi1 pad 10: (no net) -> Net-(esp_spi1-Pin_10)
- esp_spi1 pad 11: (no net) -> Net-(esp_spi1-Pin_11)
- esp_spi1 pad 12: (no net) -> Net-(esp_spi1-Pin_12)
- esp_spi1 pad 2: (no net) -> Net-(esp_spi1-Pin_2)
- esp_spi1 pad 3: (no net) -> Net-(esp_spi1-Pin_3)
- esp_spi1 pad 4: (no net) -> Net-(esp_spi1-Pin_4)
- esp_spi1 pad 5: (no net) -> Net-(esp_spi1-Pin_5)
- esp_spi1 pad 6: (no net) -> Net-(esp_spi1-Pin_6)
- esp_spi1 pad 7: (no net) -> Net-(esp_spi1-Pin_7)
- esp_spi1 pad 8: (no net) -> Net-(esp_spi1-Pin_8)
- esp_spi1 pad 9: (no net) -> Net-(esp_spi1-Pin_9)
- lora0 pad 1: (no net) -> Net-(esp_spi1-Pin_1)
- lora0 pad 10: (no net) -> Net-(esp_spi1-Pin_10)
- lora0 pad 11: (no net) -> Net-(esp_spi1-Pin_11)
- lora0 pad 12: (no net) -> Net-(esp_spi1-Pin_12)
- lora0 pad 2: (no net) -> Net-(esp_spi1-Pin_2)
- lora0 pad 3: (no net) -> Net-(esp_spi1-Pin_3)
- lora0 pad 4: (no net) -> Net-(esp_spi1-Pin_4)
- lora0 pad 5: (no net) -> Net-(esp_spi1-Pin_5)
- lora0 pad 6: (no net) -> Net-(esp_spi1-Pin_6)
- lora0 pad 7: (no net) -> Net-(esp_spi1-Pin_7)
- lora0 pad 8: (no net) -> Net-(esp_spi1-Pin_8)
- lora0 pad 9: (no net) -> Net-(esp_spi1-Pin_9)
Routing:
- net (no net): track 0.00 -> 97.2 mm, vias 4 -> 12
- net Net-(esp_spi1-Pin_10): track 0.00 -> 28.0 mm
- net Net-(esp_spi1-Pin_8): track 0.00 -> 27.6 mm
- net Net-(esp_spi1-Pin_12): track 0.00 -> 27.2 mm
- net esp_rst: track 0.00 -> 26.8 mm, vias 0 -> 2
- net esp_boot: track 0.00 -> 26.2 mm, vias 0 -> 1
- net Net-(J2-D-): track 24.6 -> 0.00 mm, vias 2 -> 0
- net Net-(J2-D+): track 24.4 -> 0.00 mm, vias 2 -> 0
- net Net-(J2-GND): track 24.3 -> 0.00 mm, vias 2 -> 0
- net Net-(J2-VBUS): track 23.9 -> 0.00 mm, vias 2 -> 0
- net Net-(esp_spi1-Pin_6): track 0.00 -> 23.3 mm
- net Net-(esp_spi1-Pin_4): track 0.00 -> 20.5 mm
- net Net-(esp_spi1-Pin_2): track 0.00 -> 19.5 mm
- net unconnected-(esp_comm1-Pin_4-Pad4): track 19.3 -> 0.00 mm, vias 1 -> 0
- net unconnected-(esp_comm1-Pin_3-Pad3): track 18.3 -> 0.00 mm, vias 1 -> 0
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Other:
- board text added: "bat0"
- board text added: "bat1"
- board text added: "boot/rst"
- board text added: "usb"
