File: board_cad/novex_rasp_hat/novex_rasp_hat.kicad_sch (KiCad schematic)
At the start: 17 parts, among them J1 GPIO, J2 USB_A, U1 CAT24C256

Commit message: CAD Novex Board Update v0.12
Parts:
- removed esp_uart_0: Conn_01x04, Connector_PinHeader_1.27mm:PinHeader_1x04_P1.27mm_Vertical, symbol Connector_Generic:Conn_01x04
- added C2, C3: C, symbol Device:C
- added C4: 100nF, symbol Device:C
- added C5: 10 uF, symbol Device:C
- added ESP_USB1: Conn_01x02, symbol Connector_Generic:Conn_01x02
- added L1: 1.5uH, symbol Device:L
- added Q1: 2N7002, Package_TO_SOT_SMD:SOT-23, symbol Transistor_FET:2N7002
- added R3: 12k, symbol Device:R
- added R4: 10k, symbol Device:R
- added R5: 1k, symbol Device:R
- added R6: 100k, symbol Device:R
- added U2: USB2514B_Bi, Package_DFN_QFN:QFN-36-1EP_6x6mm_P0.5mm_EP3.7x3.7mm, symbol Interface_USB:USB2514B_Bi
- added U3: TPS63031DSK, Package_SON:WSON-10-1EP_2.5x2.5mm_P0.5mm_EP1.2x2mm, symbol Regulator_Switching:TPS63031DSK
- added U_MCU: STM32C011F6Px, Package_SO:TSSOP-20_4.4x6.5mm_P0.65mm, symbol MCU_ST_STM32C0:STM32C011F6Px
- added Y1: 24Mhz, symbol Device:Crystal
- added bat0+, bat0-, bat1+, bat1-: TestPoint, Connector_Wire:SolderWire-0.127sqmm_1x01_D0.48mm_OD1mm, symbol Connector:TestPoint
- renumbered TP2 to D+, TP3 to D-, TP4 to GND, TP1 to VBUS, esp_spi to esp_spi1
Connections:
- net GPIO17 is gone; now on net esp_rst: J1.11 (Pin_11)
- net GPIO27 is gone; now on net esp_boot: J1.13 (Pin_13)
- net +3V3: now also R4.1, U2.10 (VDDA33), U2.15 (VDD33), U2.23 (VDD33), U2.29 (VDDA33), U2.36 (VDDA33)
- net GND: now also C2.1, C3.2, C4.2, Q1.2 (S), R3.2, R6.1, U2.37 (VSS), U3.11 (PGND), U3.3 (PGND), U3.7 (PS/SYNC), U3.9 (GND), U_MCU.5 (VSS)
- net esp_boot: now reaches esp_comm1.3 (Pin_3)
- net esp_rst: now reaches esp_comm1.4 (Pin_4)
- net RPI_INPUT_VBUS: now reaches J2.1 (VBUS), VBUS.1
- net RPI_INPUT_GND: now reaches GND.1, J2.4 (GND)
- net at J2.2 (D-): now also U2.1 (USBDM_DN1/PRT_DIS_M1); no longer D-.1
- net at J2.3 (D+): now also U2.2 (USBDP_DN1/PRT_DIS_P1); no longer D+.1
- net GPIO14/TXD0 renamed STM32_RX
- net STM32_RX: now also U_MCU.1 (PB7)
- net GPIO15/RXD0 renamed STM32_TX
- net STM32_TX: now also U_MCU.20 (PB6)
- net GPIO23 renamed STM32_SWDIO
- net STM32_SWDIO: now also U_MCU.18 (PA13)
- net GPIO24 renamed STM32_SWCLK
- net STM32_SWCLK: now also U_MCU.19 (PA14)
- net GPIO25 renamed STM32_RST
- net STM32_RST: now also U_MCU.6 (PF2)
- new net: L1.1, U3.4 (L1)
- new net: L1.2, U3.2 (L2)
- new net: ESP_USB1.1 (Pin_1), U2.3 (USBDM_DN2/PRT_DIS_M2)
- new net: ESP_USB1.2 (Pin_2), U2.4 (USBDP_DN2/PRT_DIS_P2)
- new net: Q1.1 (G), R5.2, R6.2
- new net: Q1.3 (D), R4.2, U2.26 (RESET_N)
- new net: C2.2, U2.33 (XTALIN/CLKIN), Y1.1
- new net: R3.1, U2.35 (RBIAS)
- new net: C3.1, U2.32 (XTALOUT), Y1.2
- new net +3V3_AON: C4.1, U3.1 (VOUT), U_MCU.4 (VDD)
- new net BAT_SELECTED: U3.5 (VIN), U3.6 (EN), U3.8 (VINA)
- new net RPI_INPUT_D+: D+.1, U2.31 (USBDP_UP)
- new net RPI_INPUT_D-: D-.1, U2.30 (USBDM_UP)
- new net USB_RESET_CTRL: R5.1, U_MCU.7 (PA0)
Other:
- note added: "POWER"
- note added: "RPI"
- note added: "USB"
- note added: "boot"
- note added: "rst"
- company: (none) -> xisolatedev
- title: (none) -> Novex uHAT v1
- moved on the sheet: D+, D-, GND, J2, VBUS, esp_comm1, esp_spi1, fc_conn1, lora0, sensor0
